File: temperature-sensors.kicad_pcb (KiCad board)
At the start: 4 copper layers, 60 parts, among them J1 Conn_01x03, J2 USB_C_Receptacle_PowerOnly_6P, J3 Conn_01x02, J4 Conn_01x04, Q1 AO3401A, Q2 AO3401A, Q3 AO3401A, SW1 SW_Push, SW2 SW_SPST, U1 nRF52840-QFXX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

Commit message: the pcb is pcb'd idkkkk
Parts:
- removed REF**: TPS63051-QFN-12-HotRod, temp-sensors:TPS63051-QFN-12-HotRod
- added C21: 1nF, Capacitor_SMD:C_0603_1608Metric, F.Cu at (140.9, 107.3)
- added C22: 10pF, Capacitor_SMD:C_0603_1608Metric, F.Cu at (138.0, 107.3)
- added C23: 10uF, Capacitor_SMD:C_0603_1608Metric, F.Cu at (135.0, 107.3)
- added H1: MountingHole, MountingHole:MountingHole_2.2mm_M2_ISO7380, F.Cu at (141.3, 113.7)
- added H2: MountingHole, MountingHole:MountingHole_2.2mm_M2_ISO7380, F.Cu at (117.0, 114.6)
- added H3: MountingHole, MountingHole:MountingHole_2.2mm_M2_ISO7380, F.Cu at (140.9, 82.3)
- added L5: 1.5uH, Inductor_SMD:L_1008_2520Metric, F.Cu at (135.9, 104.1)
- added R10: 560k, Resistor_SMD:R_0603_1608Metric, F.Cu at (135.0, 108.7)
- added R11: 180k, Resistor_SMD:R_0603_1608Metric, F.Cu at (138.0, 108.7)
- added R12: 1M, Resistor_SMD:R_0603_1608Metric, F.Cu at (141.7, 105.1)
- J4: value Conn_01x04 -> Conn_01x03; footprint Connector_JST:JST_PH_S4B-PH-SM4-TB_1x04-1MP_P2.00mm_Horizontal -> Connector_JST:JST_PH_S3B-PH-SM4-TB_1x03-1MP_P2.00mm_Horizontal
- R7: value 100k -> 1M
- U3: value AMS1117-3.3 -> ~; footprint Package_TO_SOT_SMD:SOT-223-3_TabPin2 -> temp-sensors:TPS63051-QFN-12-HotRod
- moved U1 58.6 mm to (125.9, 99.8), turned to -90 degrees
- moved C20 47.7 mm to (134.2, 96.7), turned to 90 degrees
- moved SW1 46.2 mm to (102.8, 114.8), turned to 180 degrees
- moved C2 46.0 mm to (122.8, 114.0), turned to 180 degrees
- moved C1 45.3 mm to (122.8, 110.7), turned to 180 degrees
- moved C6 44.9 mm to (131.0, 97.6)
- moved C12 43.9 mm to (123.7, 104.9), turned to -90 degrees
- moved C3 42.7 mm to (133.2, 102.7), turned to -90 degrees
- moved Q1 42.5 mm to (141.8, 94.6), turned to 180 degrees
- moved C13 41.6 mm to (131.0, 102.0)
- moved C11 41.2 mm to (120.8, 99.2), turned to 180 degrees
- moved Q3 40.7 mm to (140.1, 101.2)
- moved Q2 40.7 mm to (140.1, 96.9)
- moved C10 40.1 mm to (131.0, 103.5)
- moved C9 39.8 mm to (131.0, 100.6)
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Connections:
- net Net-(U1-P0.00) renamed /32768+
- net Net-(U1-P0.01) renamed /32768-
- net Net-(U1-XC1) renamed /32M+
- net Net-(U1-XC2) renamed /32M-
- J4 pad 2: /RESET -> /SWDCLK
- J4 pad 3: /SWDCLK -> /SWDIO
- R3 pad 1: GND -> Net-(U2-PROG)
- U2 pad 6: GND -> Net-(U2-PROG)
- U3 pad 1: GND -> Net-(U3-L1)
- U3 pad 2: +3V3 -> GND
- U3 pad 3: Net-(D7-K) -> Net-(U3-L2)
Routing:
- net GND: track 0.00 -> 55.1 mm, vias 0 -> 48
- net VBUS: track 0.00 -> 49.5 mm
- net /ENABLE_3V3_ON_BATT: track 0.00 -> 42.8 mm, vias 0 -> 3
- net /CONN_BATT: track 0.00 -> 41.7 mm, vias 0 -> 7
- net VDD: track 0.00 -> 41.6 mm, vias 0 -> 7
- net /SWDCLK: track 0.00 -> 39.1 mm, vias 0 -> 2
- net /SWDIO: track 0.00 -> 30.1 mm, vias 0 -> 2
- net /RESET: track 0.00 -> 26.5 mm
- net +3V3: track 0.00 -> 18.2 mm
- net /UART_RXD: track 0.00 -> 16.4 mm
- net Net-(U1-DEC4): track 0.00 -> 16.4 mm, vias 0 -> 2
- net /UART_TXD: track 0.00 -> 15.3 mm, vias 0 -> 2
- net /TMP_SENSE: track 0.00 -> 14.5 mm, vias 0 -> 2
- net Net-(U1-ANT): track 0.00 -> 11.0 mm
- net /32M-: track 0.00 -> 8.79 mm
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- added copper zone on In4.Cu, net /CONN_BATT
- added copper zone on F.Cu, net GND
- added copper zone on In1.Cu, net GND
- added copper zone on B.Cu, net VDD
Other:
- board outline added: 45 x 48 mm
- copper layers 4 -> 6

Commit message: add BOM and images and yeag
Parts:
- C16, C17: value ?pF -> 15pF
- C20: footprint Capacitor_SMD:C_0603_1608Metric -> Capacitor_SMD:C_0805_2012Metric
- C3, C4: value ?pF -> 20pF
- moved C20 0.31 mm to (133.9, 96.8)
Routing:
- net GND: track 55.1 -> 54.1 mm, vias 48 -> 47
- net VDD: track 41.6 -> 42.2 mm
Changed lines of the file:
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@@
 		)
 	)
-	(footprint "Capacitor_SMD:C_0603_1608Metric"
+	(footprint "Capacitor_SMD:C_0805_2012Metric"
 		(layer "F.Cu")
-		(at 134.19 96.705 90)
-		(descr "Capacitor SMD 0603 (1608 Metric), square (rectangular) end terminal, IPC-7351 nominal, (Body size source: IPC-SM-782 page 76, https://www.pcb-3d.com/wordpress/wp-content/uploads/ipc-sm-782a_amendment_1_and_2.pdf)")
+		(at 133.9 96.8 90)
+		(descr "Capacitor SMD 0805 (2012 Metric), square (rectangular) end terminal, IPC-7351 nominal, (Body size source: IPC-SM-782 page 76, https://www.pcb-3d.com/wordpress/wp-content/uploads/ipc-sm-782a_amendment_1_and_2.pdf, https://docs.google.com/spreadsheets/d/1BsfQQcO9C6DZCsRaXUlFlo91Tg2WpOkGARC1WS5S8t0/edit?usp=sharing)")
 		(tags "capacitor")
 		(property "Reference" "C20"
-			(at 0 -1.43 90)
+			(at 0 -1.68 90)
 			(layer "F.SilkS")
 			(effects
@@
 		)
 		(property "Value" "100uF"
-			(at 0 1.43 90)
+			(at 0 1.68 90)
 			(layer "F.Fab")
 			(effects
@@
 		(duplicate_pad_numbers_are_jumpers no)
 		(fp_line
-			(start -0.14058 -0.51)
-			(end 0.14058 -0.51)
+			(start -0.261252 -0.735)
+			(end 0.261252 -0.735)
 			(stroke
 				(width 0.12)
@@
 		)
 		(fp_line
-			(start -0.14058 0.51)
-			(end 0.14058 0.51)
+			(start -0.261252 0.735)
+			(end 0.261252 0.735)
 			(stroke
 				(width 0.12)
@@
 		)
 		(fp_rect
-			(start -1.48 -0.73)
-			(end 1.48 0.73)
+			(start -1.7 -0.98)
+			(end 1.7 0.98)
 			(stroke
 				(width 0.05)
@@
 		)
 		(fp_rect
-			(start -0.8 -0.4)
-			(end 0.8 0.4)
+			(start -1 -0.625)
+			(end 1 0.625)
 			(stroke
 				(width 0.1)
@@
 			(effects
 				(font
-					(size 0.4 0.4)
-					(thickness 0.06)
+					(size 0.5 0.5)
+					(thickness 0.08)
 				)
 			)
 		)
 		(pad "1" smd roundrect
-			(at -0.775 0 90)
-			(size 0.9 0.95)
+			(at -0.95 0 90)
+			(size 1 1.45)
 			(layers "F.Cu" "F.Mask" "F.Paste")
 			(roundrect_rratio 0.25)
@@
 		)
 		(pad "2" smd roundrect
-			(at 0.775 0 90)
-			(size 0.9 0.95)
+			(at 0.95 0 90)
+			(size 1 1.45)
 			(layers "F.Cu" "F.Mask" "F.Paste")
 			(roundrect_rratio 0.25)
@@
 		)
 		(embedded_fonts no)
-		(model "${KICAD10_3DMODEL_DIR}/Capacitor_SMD.3dshapes/C_0603_1608Metric.step"
+		(model "${KICAD10_3DMODEL_DIR}/Capacitor_SMD.3dshapes/C_0805_2012Metric.step"
 			(offset
 				(xyz 0 0 0)
@@
 			)
 		)
-		(property "Value" "?pF"
+		(property "Value" "15pF"
 			(at 0 1.43 0)
 			(layer "F.Fab")
@@
 			)
 		)
-		(property "Value" "?pF"
+		(property "Value" "15pF"
 			(at 0 1.43 90)
 			(layer "F.Fab")
@@
 			)
 		)
-		(property "Value" "?pF"
+		(property "Value" "20pF"
 			(at 0 1.43 0)
 			(layer "F.Fab")
@@
 				(name "A")
 				(pins "35" "36" "2" "3" "29" "30" "40" "39" "4" "5" "7" "13" "14" "15"
-					"18" "19" "20" "21" "22" "23" "41" "42" "43" "44" "8" "38" "28" "17"
-					"25" "12" "37" "48" "32" "45" "49" "47" "1" "34" "46" "33" "31" "24"
+					"18" "19" "20" "21" "22" "23" "41" "42" "43" "44" "8" "38" "28" "48"
+					"37" "12" "17" "25" "32" "49" "45" "47" "1" "34" "46" "33" "31" "24"
 					"11" "10" "9" "6" "16" "27" "26"
 				)
@@
 			)
 		)
-		(property "Value" "?pF"
+		(property "Value" "20pF"
 			(at 0 1.43 90)
 			(layer "F.Fab")
@@
 	)
 	(segment
-		(start 134.19 97.48)
-		(end 135.465 97.48)
-		(width 0.2)
-		(layer "F.Cu")
-		(net "VDD")
-	)
-	(segment
 		(start 121.025 107.112107)
 		(end 122.072893 108.16)
@@
 	)
 	(segment
+		(start 135.47 96.815)
+		(end 134.835 96.815)
+		(width 0.2)
+		(layer "F.Cu")
+		(net "VDD")
+	)
+	(segment
 		(start 122.072893 108.16)
 		(end 122.487107 108.16)
@@
 	)
 	(segment
+		(start 134.835 96.815)
+		(end 133.9 97.75)
+		(width 0.2)
+		(layer "F.Cu")
+		(net "VDD")
+	)
+	(segment
 		(start 120.325 103.1)
 		(end 120.325 104.7125)
@@
 	)
 	(via
-		(at 130.19 102.03)
+		(at 133.9 97.75)
 		(size 0.6)
 		(drill 0.3)
@@
 	)
 	(via
-		(at 134.19 97.48)
+		(at 130.19 102.03)
 		(size 0.6)
 		(drill 0.3)
@@
 	)
 	(segment
-		(start 137.3175 94.295)
-		(end 136.1625 94.295)
-		(width 0.2)
-		(layer "F.Cu")
-		(net "GND")
-	)
-	(segment
 		(start 139.47 105.193419)
 		(end 138.736595 104.460014)
@@
 	)
 	(segment
-		(start 131.4525 94.77)
-		(end 131.4525 94.295)
+		(start 134.6075 95.85)
+		(end 135.9625 94.495)
 		(width 0.2)
 		(layer "F.Cu")
@@
 	)
 	(segment
-		(start 134.5275 95.93)
-		(end 135.96125 94.49625)
+		(start 131.4525 94.295)
+		(end 131.4525 94.5525)
 		(width 0.2)
 		(layer "F.Cu")
@@
 	)
 	(segment
-		(start 134.19 95.93)
-		(end 132.6125 95.93)
-		(width 0.2)
-		(layer "F.Cu")
-		(net "GND")
-	)
-	(segment
 		(start 129.86 94.74)
 		(end 131.29 96.17)
@@
 	)
 	(segment
+		(start 133.9 95.85)
+		(end 134.6075 95.85)
+		(width 0.2)
+		(layer "F.Cu")
+		(net "GND")
+	)
+	(segment
 		(start 139.47 105.895)
 		(end 139.47 105.193419)
@@
 	)
 	(segment
+		(start 131.4525 94.5525)
+		(end 132.75 95.85)
+		(width 0.2)
+		(layer "F.Cu")
+		(net "GND")
+	)
+	(segment
 		(start 113.895 86.86)
 		(end 114.355 87.32)
@@
 	)
 	(segment
-		(start 132.6125 95.93)
-		(end 131.4525 94.77)
-		(width 0.2)
-		(layer "F.Cu")
-		(net "GND")
-	)
-	(segment
 		(start 138.701609 104.495)
 		(end 138.736595 104.460014)
@@
 	)
 	(segment
+		(start 132.75 95.85)
+		(end 133.9 95.85)
+		(width 0.2)
+		(layer "F.Cu")
+		(net "GND")
+	)
+	(segment
 		(start 112.405 85.37)
 		(end 113.895 86.86)
@@
 	)
 	(via
-		(at 135.96125 94.49625)
-		(size 0.6)
-		(drill 0.3)
-		(layers "F.Cu" "B.Cu")
-		(net "GND")
-	)
-	(via
 		(at 133.62 92.065)
 		(size 0.4)
@@
 	)
 	(via
-		(at 134.19 95.93)
-		(size 0.6)
-		(drill 0.3)
-		(layers "F.Cu" "B.Cu")
-		(net "GND")
-	)
-	(via
 		(at 120.28 111.63)
 		(size 0.4)
@@
 		(size 0.6)
 		(drill 0.3)
+		(layers "F.Cu" "B.Cu")
+		(net "GND")
+	)
+	(via
+		(at 133.9 95.85)
+		(size 0.6)
+		(drill 0.3)
